File: hardware/pcb/Power.sch (KiCad schematic (older format))
At the start: 28 parts, among them CON201 USB-MICRO-B, P202 CONN_01X02, U201 FT232RQ, U202 MCP1700T-3302E/TT

Commit message: Opened and saved with KiCad 4.0.5
Parts:
- D203, D204, D205: symbol LED -> LED-RESCUE-CentralCommand
Changed lines of the file:
@@
 EESchema Schematic File Version 2
+LIBS:CentralCommand-rescue
 LIBS:power
 LIBS:device
@@
 VCC
 $Comp
-L LED D203
+L LED-RESCUE-CentralCommand D203
 U 1 1 56C6507B
 P 5100 4900
@@
 $EndComp
 $Comp
-L LED D204
+L LED-RESCUE-CentralCommand D204
 U 1 1 56C650D3
 P 5350 5050
@@
 $EndComp
 $Comp
-L LED D205
+L LED-RESCUE-CentralCommand D205
 U 1 1 56CC1A90
 P 5950 2100
