File: hardware/pcb/Power.sch (KiCad schematic (older format))
At the start: 28 parts, among them CON201 USB-MICRO-B, P202 CONN_01X02, U201 FT232RQ, U202 MCP1700T-3302E/TT

Commit message: CC56
Parts:
- C201, C202, C204: footprint Capacitors_SMD:C_0805 -> CE_Capacitor:C_0805
- C203, C205, C206: footprint Capacitors_SMD:C_1210 -> CE_Capacitor:C_1210
- CON201: footprint pcb:MICRO_B_CONN_10118193-0001LF -> CE_Connector:MICRO_B_CONN_10118193-0001LF
- D203, D204, D205: footprint LEDs:LED_0805 -> CE_Diode:LED_0805
- FB201: footprint Inductors_NEOSID:Neosid_Inductor_SM1206 -> CE_Inductor:Neosid_Inductor_SM1206
- JP201: footprint Pin_Headers:Pin_Header_Straight_1x03 -> CE_Connector:Pin_Header_Straight_1x03
- P202: footprint Pin_Headers:Pin_Header_Straight_1x02 -> CE_Connector:Pin_Header_Straight_1x02
- R201, R202, R203, R204, R205, R206, R207, R208, R209, R210, R211: footprint Resistors_SMD:R_0805 -> CE_Resistor:R_0805
- U201: footprint Housings_DFN_QFN:QFN-32-1EP_5x5mm_Pitch0.5mm -> CE_IC:QFN-32-1EP_5x5mm_Pitch0.5mm
- U202: footprint pcb:SOT-23 -> CE_Regulator:SOT-23
Changed lines of the file:
@@
 F 0 "U202" H 4600 1950 60  0000 C CNN
 F 1 "MCP1700T-3302E/TT" H 4600 1800 60  0000 C CNN
-F 2 "pcb:SOT-23" H 4600 1750 60  0001 C CNN
+F 2 "CE_Regulator:SOT-23" H 4600 1750 60  0001 C CNN
 F 3 "" H 4600 1750 60  0000 C CNN
 F 4 "MCP1700T-3302E/TT" H 4600 1750 60  0001 C CNN "MPN"
@@
 F 0 "C205" H 3775 1900 50  0000 L CNN
 F 1 "10uf" H 3775 1700 50  0000 L CNN
-F 2 "Capacitors_SMD:C_1210" H 3788 1650 50  0001 C CNN
+F 2 "CE_Capacitor:C_1210" H 3788 1650 50  0001 C CNN
 F 3 "" H 3750 1800 50  0000 C CNN
 	1    3750 1800
@@
 F 0 "C206" H 5425 1900 50  0000 L CNN
 F 1 "10uf" H 5425 1700 50  0000 L CNN
-F 2 "Capacitors_SMD:C_1210" H 5438 1650 50  0001 C CNN
+F 2 "CE_Capacitor:C_1210" H 5438 1650 50  0001 C CNN
 F 3 "" H 5400 1800 50  0000 C CNN
 	1    5400 1800
@@
 F 0 "U201" H 3700 4150 60  0000 C CNN
 F 1 "FT232RQ" H 3700 4650 60  0000 C CNN
-F 2 "Housings_DFN_QFN:QFN-32-1EP_5x5mm_Pitch0.5mm" H 3800 4200 60  0001 C CNN
+F 2 "CE_IC:QFN-32-1EP_5x5mm_Pitch0.5mm" H 3800 4200 60  0001 C CNN
 F 3 "" H 3800 4200 60  0000 C CNN
 F 4 "FT232RQ-REEL" H 3700 4600 60  0001 C CNN "MPN"
@@
 F 0 "FB201" H 2000 3950 50  0000 C CNN
 F 1 "FILTER" H 2100 3700 50  0000 C CNN
-F 2 "Inductors_NEOSID:Neosid_Inductor_SM1206" H 2100 3800 50  0001 C CNN
+F 2 "CE_Inductor:Neosid_Inductor_SM1206" H 2100 3800 50  0001 C CNN
 F 3 "http://search.murata.co.jp/Ceramy/image/img/PDF/ENG/L0110S0100BLM41P.pdf" H 2100 3800 50  0001 C CNN
 F 4 "BLM41PG471SN1L" H 2100 3800 60  0001 C CNN "MPN"
@@
 F 0 "C201" H 1675 3600 50  0000 L CNN
 F 1 "10nf" H 1675 3400 50  0000 L CNN
-F 2 "Capacitors_SMD:C_0805" H 1688 3350 50  0001 C CNN
+F 2 "CE_Capacitor:C_0805" H 1688 3350 50  0001 C CNN
 F 3 "" H 1650 3500 50  0000 C CNN
 	1    1650 3500
@@
 F 0 "P202" H 900 1750 50  0000 C CNN
 F 1 "CONN_01X02" V 1000 1600 50  0000 C CNN
-F 2 "Pin_Headers:Pin_Header_Straight_1x02" H 900 1600 50  0001 C CNN
+F 2 "CE_Connector:Pin_Header_Straight_1x02" H 900 1600 50  0001 C CNN
 F 3 "" H 900 1600 50  0000 C CNN
 	1    900  1600
@@
 F 0 "C204" H 2625 5600 50  0000 L CNN
 F 1 "100nf" H 2625 5400 50  0000 L CNN
-F 2 "Capacitors_SMD:C_0805" H 2638 5350 50  0001 C CNN
+F 2 "CE_Capacitor:C_0805" H 2638 5350 50  0001 C CNN
 F 3 "" H 2600 5500 50  0000 C CNN
 	1    2600 5500
@@
 F 0 "C202" H 2125 3100 50  0000 L CNN
 F 1 "100nf" H 2125 2900 50  0000 L CNN
-F 2 "Capacitors_SMD:C_0805" H 2138 2850 50  0001 C CNN
+F 2 "CE_Capacitor:C_0805" H 2138 2850 50  0001 C CNN
 F 3 "" H 2100 3000 50  0000 C CNN
 	1    2100 3000
@@
 F 0 "C203" H 2425 3100 50  0000 L CNN
 F 1 "4.7uf" H 2425 2900 50  0000 L CNN
-F 2 "Capacitors_SMD:C_1210" H 2438 2850 50  0001 C CNN
+F 2 "CE_Capacitor:C_1210" H 2438 2850 50  0001 C CNN
 F 3 "" H 2400 3000 50  0000 C CNN
 	1    2400 3000
@@
 F 0 "R201" V 2880 4900 50  0000 C CNN
 F 1 "0" V 2800 4900 50  0000 C CNN
-F 2 "Resistors_SMD:R_0805" V 2730 4900 50  0001 C CNN
+F 2 "CE_Resistor:R_0805" V 2730 4900 50  0001 C CNN
 F 3 "" H 2800 4900 50  0000 C CNN
 	1    2800 4900
@@
 F 0 "D203" H 5100 5000 50  0000 C CNN
 F 1 "LED_GREEN" H 5100 4800 50  0000 C CNN
-F 2 "LEDs:LED_0805" H 5100 4900 50  0001 C CNN
+F 2 "CE_Diode:LED_0805" H 5100 4900 50  0001 C CNN
 F 3 "" H 5100 4900 50  0000 C CNN
 F 4 "150080GS75000" H 5100 4900 60  0001 C CNN "MPN"
@@
 F 0 "D204" H 5350 5150 50  0000 C CNN
 F 1 "LED_YELLOW" H 5350 4950 50  0000 C CNN
-F 2 "LEDs:LED_0805" H 5350 5050 50  0001 C CNN
+F 2 "CE_Diode:LED_0805" H 5350 5050 50  0001 C CNN
 F 3 "" H 5350 5050 50  0000 C CNN
 F 4 "150080YS75000" H 5350 5050 60  0001 C CNN "MPN"
@@
 F 0 "R208" V 5680 4900 50  0000 C CNN
 F 1 "270" V 5600 4900 50  0000 C CNN
-F 2 "Resistors_SMD:R_0805" V 5530 4900 50  0001 C CNN
+F 2 "CE_Resistor:R_0805" V 5530 4900 50  0001 C CNN
 F 3 "" H 5600 4900 50  0000 C CNN
 	1    5600 4900
@@
 F 0 "R209" V 6030 5050 50  0000 C CNN
 F 1 "270" V 5950 5050 50  0000 C CNN
-F 2 "Resistors_SMD:R_0805" V 5880 5050 50  0001 C CNN
+F 2 "CE_Resistor:R_0805" V 5880 5050 50  0001 C CNN
 F 3 "" H 5950 5050 50  0000 C CNN
 	1    5950 5050
@@
 F 0 "R204" V 4880 4000 50  0000 C CNN
 F 1 "NOP" V 4800 4000 50  0000 C CNN
-F 2 "Resistors_SMD:R_0805" V 4730 4000 50  0001 C CNN
+F 2 "CE_Resistor:R_0805" V 4730 4000 50  0001 C CNN
 F 3 "" H 4800 4000 50  0000 C CNN
 	1    4800 4000
@@
 F 0 "R206" V 5130 4150 50  0000 C CNN
 F 1 "NOP" V 5050 4150 50  0000 C CNN
-F 2 "Resistors_SMD:R_0805" V 4980 4150 50  0001 C CNN
+F 2 "CE_Resistor:R_0805" V 4980 4150 50  0001 C CNN
 F 3 "" H 5050 4150 50  0000 C CNN
 	1    5050 4150
@@
 F 0 "R203" V 4180 5950 50  0000 C CNN
 F 1 "0" V 4100 5950 50  0000 C CNN
-F 2 "Resistors_SMD:R_0805" V 4030 5950 50  0001 C CNN
+F 2 "CE_Resistor:R_0805" V 4030 5950 50  0001 C CNN
 F 3 "" H 4100 5950 50  0000 C CNN
 	1    4100 5950
@@
 F 0 "R205" V 4930 3700 50  0000 C CNN
 F 1 "0" V 4850 3700 50  0000 C CNN
-F 2 "Resistors_SMD:R_0805" V 4780 3700 50  0001 C CNN
+F 2 "CE_Resistor:R_0805" V 4780 3700 50  0001 C CNN
 F 3 "" H 4850 3700 50  0000 C CNN
 	1    4850 3700
@@
 F 0 "R207" V 5180 3850 50  0000 C CNN
 F 1 "0" V 5100 3850 50  0000 C CNN
-F 2 "Resistors_SMD:R_0805" V 5030 3850 50  0001 C CNN
+F 2 "CE_Resistor:R_0805" V 5030 3850 50  0001 C CNN
 F 3 "" H 5100 3850 50  0000 C CNN
 	1    5100 3850
@@
 F 0 "R202" V 2930 5300 50  0000 C CNN
 F 1 "0" V 2850 5300 50  0000 C CNN
-F 2 "Resistors_SMD:R_0805" V 2780 5300 50  0001 C CNN
+F 2 "CE_Resistor:R_0805" V 2780 5300 50  0001 C CNN
 F 3 "" H 2850 5300 50  0000 C CNN
 	1    2850 5300
@@
 F 0 "CON201" H 750 4350 50  0000 C CNN
 F 1 "USB-MICRO-B" H 900 3650 50  0000 C CNN
-F 2 "pcb:MICRO_B_CONN_10118193-0001LF" H 1050 3900 50  0001 C CNN
+F 2 "CE_Connector:MICRO_B_CONN_10118193-0001LF" H 1050 3900 50  0001 C CNN
 F 3 "" H 1050 3900 50  0000 C CNN
 F 4 "10118193-0001LF" H 1050 4000 60  0001 C CNN "MPN"
@@
 F 0 "R210" V 2180 4200 50  0000 C CNN
 F 1 "NOP" V 2100 4200 50  0000 C CNN
-F 2 "Resistors_SMD:R_0805" V 2030 4200 50  0001 C CNN
+F 2 "CE_Resistor:R_0805" V 2030 4200 50  0001 C CNN
 F 3 "" H 2100 4200 50  0000 C CNN
 	1    2100 4200
@@
 F 0 "D205" H 5950 2200 50  0000 C CNN
 F 1 "LED_BLUE" H 5950 2000 50  0000 C CNN
-F 2 "LEDs:LED_0805" H 5950 2100 50  0001 C CNN
+F 2 "CE_Diode:LED_0805" H 5950 2100 50  0001 C CNN
 F 3 "" H 5950 2100 50  0000 C CNN
 F 4 "150080BS75000" H 5950 2100 60  0001 C CNN "MPN"
@@
 F 0 "R211" V 5880 1750 50  0000 C CNN
 F 1 "270" V 5800 1750 50  0000 C CNN
-F 2 "Resistors_SMD:R_0805" V 5730 1750 50  0001 C CNN
+F 2 "CE_Resistor:R_0805" V 5730 1750 50  0001 C CNN
 F 3 "" H 5800 1750 50  0000 C CNN
 	1    5800 1750
@@
 F 0 "JP201" H 2750 1450 50  0000 L CNN
 F 1 "JUMPER3" H 2700 1650 50  0000 C BNN
-F 2 "Pin_Headers:Pin_Header_Straight_1x03" H 2700 1550 50  0001 C CNN
+F 2 "CE_Connector:Pin_Header_Straight_1x03" H 2700 1550 50  0001 C CNN
 F 3 "" H 2700 1550 50  0000 C CNN
 	1    2700 1550

Commit message: CC56
Parts:
- D201, D202: footprint Diodes_SMD:SOD-123 -> CE_Diode:SOD-123
Changed lines of the file:
@@
 F 0 "D201" H 1550 1650 50  0000 C CNN
 F 1 "D_Schottky" H 1550 1450 50  0000 C CNN
-F 2 "Diodes_SMD:SOD-123" H 1550 1550 50  0001 C CNN
+F 2 "CE_Diode:SOD-123" H 1550 1550 50  0001 C CNN
 F 3 "" H 1550 1550 50  0000 C CNN
 F 4 "MBR0520LT1G" H 1550 1550 60  0001 C CNN "MPN"
@@
 F 0 "D202" H 2700 3500 50  0000 C CNN
 F 1 "D_Schottky" H 2700 3300 50  0000 C CNN
-F 2 "Diodes_SMD:SOD-123" H 2700 3400 50  0001 C CNN
+F 2 "CE_Diode:SOD-123" H 2700 3400 50  0001 C CNN
 F 3 "" H 2700 3400 50  0000 C CNN
 F 4 "MBR0520LT1G" H 2700 3400 60  0001 C CNN "MPN"

Commit message: CC58
Parts:
- removed C201: 10nf, CE_Capacitor:C_0805, symbol C
- removed C202, C204: 100nf, CE_Capacitor:C_0805, symbol C
- removed C203: 4.7uf, CE_Capacitor:C_1210, symbol C
- removed C205, C206: 10uf, CE_Capacitor:C_1210, symbol C
- removed CON201: USB-MICRO-B, CE_Connector:MICRO_B_CONN_10118193-0001LF, symbol USB-MICRO-B
- removed D201, D202: D_Schottky, CE_Diode:SOD-123, symbol D_Schottky
- removed D203: LED_GREEN, CE_Diode:LED_0805, symbol LED-RESCUE-CentralCommand
- removed D204: LED_YELLOW, CE_Diode:LED_0805, symbol LED-RESCUE-CentralCommand
- removed D205: LED_BLUE, CE_Diode:LED_0805, symbol LED-RESCUE-CentralCommand
- removed FB201: FILTER, CE_Inductor:Neosid_Inductor_SM1206, symbol FILTER
- removed R201, R202, R203, R205, R207: 0, CE_Resistor:R_0805, symbol R
- removed R208, R209, R211: 270, CE_Resistor:R_0805, symbol R
- added C201: C0805C103K3RACTU, CE_Capacitor:C_0805, symbol C0805C103K3RACTU
- added C202, C204: 08055C104JAT2A, CE_Capacitor:C_0805, symbol 08055C104JAT2A
- added C203: CL21B475KOFNNNE, CE_Capacitor:C_0805, symbol CL21B475KOFNNNE
- added C205, C206: TMK325B7106KN-TR, CE_Capacitor:C_1210, symbol TMK325B7106KN-TR
- added CON201: 10118193-0001LF, CE_Connector:MICRO_B_CONN_10118193-0001LF, symbol 10118193-0001LF
- added D201, D202: MBR0520LT1G, CE_Diode:SOD-123, symbol MBR0520LT1G
- added D203: 150080GS75000, CE_Diode:LED_0805, symbol 150080GS75000
- added D204: 150080YS75000, CE_Diode:LED_0805, symbol 150080YS75000
- added D205: 150080BS75000, CE_Diode:LED_0805, symbol 150080BS75000
- added FB201: BLM41PG471SN1L, CE_Filter:Filter_SM1806, symbol BLM41PG471SN1L
- added R201, R202, R203, R205, R207: ERJ-6GEY0R00V, CE_Resistor:R_0805, symbol ERJ-6GEY0R00V
- added R208, R209, R211: RNCP0805FTD200R, CE_Resistor:R_0805, symbol RNCP0805FTD200R
Connections:
- net EXT_PWR: now also D201.1 (K)
- net GND: now also C201.1, C202.1, C203.1, C204.2, C205.2, C206.2, CON201.5 (GND), CON201.6 (SHELL1), CON201.7 (SHELL2), CON201.8 (SHELL3), CON201.9 (SHELL4), D205.1 (K), R203.2
- net PWR: now also C206.1, R211.2
- net RESET#: now also R201.1
- net RXD: now also R205.2
- net TXD: now also R207.2
- net USB_PWR: now also D202.1 (K)
- net VCC: now also C202.2, C203.2, D202.2 (A), FB201.2, R208.1, R209.1
- net at JP201.2, U202.3 (IN): now also C205.1
- net at U201.14 (USBDP): now also CON201.3 (D+)
- net at U201.15 (USBDM): now also CON201.2 (D-)
- net at U201.16 (3V3OUT): now also R202.2
- net at U201.18 (RESET#): now also R201.2
- net at U201.2 (RXD): now also R207.1
- net at U201.21 (CBUS1): now also D204.1 (K)
- net at U201.22 (CBUS0): now also D203.1 (K)
- net at U201.26 (TEST): now also R203.1
- net at U201.30 (TXD): now also R205.1
- net at P202.1 (P1): now also D201.2 (A)
- net at R210.2: now also CON201.4 (ID)
- new net: C201.2, CON201.1 (VBUS), FB201.1
- new net: D205.2 (A), R211.1
- new net: C204.1, R202.1
- new net: D203.2 (A), R208.2
- new net: D204.2 (A), R209.2
