File: hardware/pcb/CentralCommand.sch (KiCad schematic (older format))
At the start: 22 parts, among them P101 CONN_01X10, P102 CONN_01X10, P103 CONN_01X04, P104 CONN_01X04, P105 CONN_01X02, P106 CONN_01X02, P107 CONN_01X01, P108 CONN_01X01, P109 CONN_01X01, P110 CONN_01X01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

Commit message: CC56
Parts:
- C101, C102, C103, C104, C107: footprint Capacitors_SMD:C_0805 -> CE_Capacitor:C_0805
- C105, C106, C108, C109: footprint Capacitors_SMD:C_1206 -> CE_Capacitor:C_1206
- L101: footprint Inductors_NEOSID:Neosid_Inductor_SM1206 -> CE_Inductor:Neosid_Inductor_SM1206
- P101, P102: footprint Pin_Headers:Pin_Header_Straight_1x10 -> CE_Connector:Pin_Header_Straight_1x10
- P103, P104: footprint Pin_Headers:Pin_Header_Straight_1x04 -> CE_Connector:Pin_Header_Straight_1x04
- P105, P106: footprint Pin_Headers:Pin_Header_Straight_1x02 -> CE_Connector:Pin_Header_Straight_1x02
- P107, P108, P109, P110: footprint Mounting_Holes:MountingHole_3mm -> CE_MountingHole:MountingHole_3mm
- U101: footprint Housings_QFP:LQFP-48_7x7mm_Pitch0.5mm -> CE_IC:LQFP-48_7x7mm_Pitch0.5mm
- Y101: footprint pcb:Crystal_HC49_US -> CE_Crystal:Crystal_HC49_US
Changed lines of the file:
@@
 F 0 "L101" V 6150 800 50  0000 C CNN
 F 1 "10uh" V 6300 800 50  0000 C CNN
-F 2 "Inductors_NEOSID:Neosid_Inductor_SM1206" H 6200 800 50  0001 C CNN
+F 2 "CE_Inductor:Neosid_Inductor_SM1206" H 6200 800 50  0001 C CNN
 F 3 "" H 6200 800 50  0000 C CNN
 F 4 "AIML-1206-100K-T" H 6200 800 60  0001 C CNN "MPN"
@@
 F 0 "C101" H 6975 1150 50  0000 L CNN
 F 1 ".1uf" H 6975 950 50  0000 L CNN
-F 2 "Capacitors_SMD:C_0805" H 6988 900 50  0001 C CNN
+F 2 "CE_Capacitor:C_0805" H 6988 900 50  0001 C CNN
 F 3 "" H 6950 1050 50  0000 C CNN
 	1    6950 1050
@@
 F 0 "U101" V 4500 3500 60  0000 C CNN
 F 1 "STM32F030C8" V 4500 2950 60  0000 C CNN
-F 2 "Housings_QFP:LQFP-48_7x7mm_Pitch0.5mm" H 3850 3850 60  0001 C CNN
+F 2 "CE_IC:LQFP-48_7x7mm_Pitch0.5mm" H 3850 3850 60  0001 C CNN
 F 3 "" H 3850 3850 60  0000 C CNN
 F 4 "STM32F030C8T6" H 3850 3850 60  0001 C CNN "MPN"
@@
 F 0 "U101" V 4500 6150 60  0000 C CNN
 F 1 "STM32F030C8" V 4500 5600 60  0000 C CNN
-F 2 "Housings_QFP:LQFP-48_7x7mm_Pitch0.5mm" H 3850 6500 60  0001 C CNN
+F 2 "CE_IC:LQFP-48_7x7mm_Pitch0.5mm" H 3850 6500 60  0001 C CNN
 F 3 "" H 3850 6500 60  0000 C CNN
 F 4 "STM32F030C8T6" H 3850 6500 60  0001 C CNN "MPN"
@@
 F 0 "U101" V 6700 2100 60  0000 C CNN
 F 1 "STM32F030C8" V 6700 1550 60  0000 C CNN
-F 2 "Housings_QFP:LQFP-48_7x7mm_Pitch0.5mm" H 6050 2450 60  0001 C CNN
+F 2 "CE_IC:LQFP-48_7x7mm_Pitch0.5mm" H 6050 2450 60  0001 C CNN
 F 3 "" H 6050 2450 60  0000 C CNN
 F 4 "STM32F030C8T6" H 6050 2450 60  0001 C CNN "MPN"
@@
 F 0 "Y101" H 7800 1950 50  0000 C CNN
 F 1 "Crystal" H 7800 1650 50  0000 C CNN
-F 2 "pcb:Crystal_HC49_US" H 7800 1800 50  0001 C CNN
+F 2 "CE_Crystal:Crystal_HC49_US" H 7800 1800 50  0001 C CNN
 F 3 "" H 7800 1800 50  0000 C CNN
 F 4 "9C-8.000MEEJ-T" H 7800 1800 60  0001 C CNN "MPN"
@@
 F 0 "C102" H 8275 1650 50  0000 L CNN
 F 1 "18pf" H 8275 1450 50  0000 L CNN
-F 2 "Capacitors_SMD:C_0805" H 8288 1400 50  0001 C CNN
+F 2 "CE_Capacitor:C_0805" H 8288 1400 50  0001 C CNN
 F 3 "" H 8250 1550 50  0000 C CNN
 	1    8250 1550
@@
 F 0 "C103" H 8275 2150 50  0000 L CNN
 F 1 "18pf" H 8275 1950 50  0000 L CNN
-F 2 "Capacitors_SMD:C_0805" H 8288 1900 50  0001 C CNN
+F 2 "CE_Capacitor:C_0805" H 8288 1900 50  0001 C CNN
 F 3 "" H 8250 2050 50  0000 C CNN
 	1    8250 2050
@@
 F 0 "P101" H 850 2800 50  0000 C CNN
 F 1 "CONN_01X10" V 950 2250 50  0000 C CNN
-F 2 "Pin_Headers:Pin_Header_Straight_1x10" H 850 2250 50  0001 C CNN
+F 2 "CE_Connector:Pin_Header_Straight_1x10" H 850 2250 50  0001 C CNN
 F 3 "" H 850 2250 50  0000 C CNN
 	1    850  2250
@@
 F 0 "P103" H 5200 5100 50  0000 C CNN
 F 1 "CONN_01X04" V 5300 4850 50  0000 C CNN
-F 2 "Pin_Headers:Pin_Header_Straight_1x04" H 5200 4850 50  0001 C CNN
+F 2 "CE_Connector:Pin_Header_Straight_1x04" H 5200 4850 50  0001 C CNN
 F 3 "" H 5200 4850 50  0000 C CNN
 	1    5200 4850
@@
 F 0 "P104" H 5200 6250 50  0000 C CNN
 F 1 "CONN_01X04" V 5300 6000 50  0000 C CNN
-F 2 "Pin_Headers:Pin_Header_Straight_1x04" H 5200 6000 50  0001 C CNN
+F 2 "CE_Connector:Pin_Header_Straight_1x04" H 5200 6000 50  0001 C CNN
 F 3 "" H 5200 6000 50  0000 C CNN
 	1    5200 6000
@@
 F 0 "P105" H 5200 7100 50  0000 C CNN
 F 1 "CONN_01X02" V 5300 6950 50  0000 C CNN
-F 2 "Pin_Headers:Pin_Header_Straight_1x02" H 5200 6950 50  0001 C CNN
+F 2 "CE_Connector:Pin_Header_Straight_1x02" H 5200 6950 50  0001 C CNN
 F 3 "" H 5200 6950 50  0000 C CNN
 	1    5200 6950
@@
 F 0 "P102" H 900 7200 50  0000 C CNN
 F 1 "CONN_01X10" V 1000 6650 50  0000 C CNN
-F 2 "Pin_Headers:Pin_Header_Straight_1x10" H 900 6650 50  0001 C CNN
+F 2 "CE_Connector:Pin_Header_Straight_1x10" H 900 6650 50  0001 C CNN
 F 3 "" H 900 6650 50  0000 C CNN
 	1    900  6650
@@
 F 0 "P106" H 6850 5000 50  0000 C CNN
 F 1 "CONN_01X02" V 6950 4850 50  0000 C CNN
-F 2 "Pin_Headers:Pin_Header_Straight_1x02" H 6850 4850 50  0001 C CNN
+F 2 "CE_Connector:Pin_Header_Straight_1x02" H 6850 4850 50  0001 C CNN
 F 3 "" H 6850 4850 50  0000 C CNN
 	1    6850 4850
@@
 F 0 "P107" H 10350 1000 50  0000 C CNN
 F 1 "CONN_01X01" V 10450 900 50  0000 C CNN
-F 2 "Mounting_Holes:MountingHole_3mm" H 10350 900 50  0001 C CNN
+F 2 "CE_MountingHole:MountingHole_3mm" H 10350 900 50  0001 C CNN
 F 3 "" H 10350 900 50  0000 C CNN
 	1    10350 900
@@
 F 0 "P108" H 10350 1550 50  0000 C CNN
 F 1 "CONN_01X01" V 10450 1450 50  0000 C CNN
-F 2 "Mounting_Holes:MountingHole_3mm" H 10350 1450 50  0001 C CNN
+F 2 "CE_MountingHole:MountingHole_3mm" H 10350 1450 50  0001 C CNN
 F 3 "" H 10350 1450 50  0000 C CNN
 	1    10350 1450
@@
 F 0 "P110" H 10800 1550 50  0000 C CNN
 F 1 "CONN_01X01" V 10900 1450 50  0000 C CNN
-F 2 "Mounting_Holes:MountingHole_3mm" H 10800 1450 50  0001 C CNN
+F 2 "CE_MountingHole:MountingHole_3mm" H 10800 1450 50  0001 C CNN
 F 3 "" H 10800 1450 50  0000 C CNN
 	1    10800 1450
@@
 F 0 "P109" H 10800 1000 50  0000 C CNN
 F 1 "CONN_01X01" V 10900 900 50  0000 C CNN
-F 2 "Mounting_Holes:MountingHole_3mm" H 10800 900 50  0001 C CNN
+F 2 "CE_MountingHole:MountingHole_3mm" H 10800 900 50  0001 C CNN
 F 3 "" H 10800 900 50  0000 C CNN
 	1    10800 900
@@
 F 0 "C104" H 1875 1250 50  0000 L CNN
 F 1 "0.1u" H 1875 1050 50  0000 L CNN
-F 2 "Capacitors_SMD:C_0805" H 1888 1000 50  0001 C CNN
+F 2 "CE_Capacitor:C_0805" H 1888 1000 50  0001 C CNN
 F 3 "" H 1850 1150 50  0000 C CNN
 	1    1850 1150
@@
 F 0 "C105" H 2175 1250 50  0000 L CNN
 F 1 "1u" H 2175 1050 50  0000 L CNN
-F 2 "Capacitors_SMD:C_1206" H 2188 1000 50  0001 C CNN
+F 2 "CE_Capacitor:C_1206" H 2188 1000 50  0001 C CNN
 F 3 "" H 2150 1150 50  0000 C CNN
 	1    2150 1150
@@
 F 0 "C106" H 2425 1250 50  0000 L CNN
 F 1 "10u" H 2425 1050 50  0000 L CNN
-F 2 "Capacitors_SMD:C_1206" H 2438 1000 50  0001 C CNN
+F 2 "CE_Capacitor:C_1206" H 2438 1000 50  0001 C CNN
 F 3 "" H 2400 1150 50  0000 C CNN
 	1    2400 1150
@@
 F 0 "C107" H 2875 1250 50  0000 L CNN
 F 1 "0.1u" H 2875 1050 50  0000 L CNN
-F 2 "Capacitors_SMD:C_0805" H 2888 1000 50  0001 C CNN
+F 2 "CE_Capacitor:C_0805" H 2888 1000 50  0001 C CNN
 F 3 "" H 2850 1150 50  0000 C CNN
 	1    2850 1150
@@
 F 0 "C108" H 3175 1250 50  0000 L CNN
 F 1 "1u" H 3175 1050 50  0000 L CNN
-F 2 "Capacitors_SMD:C_1206" H 3188 1000 50  0001 C CNN
+F 2 "CE_Capacitor:C_1206" H 3188 1000 50  0001 C CNN
 F 3 "" H 3150 1150 50  0000 C CNN
 	1    3150 1150
@@
 F 0 "C109" H 3425 1250 50  0000 L CNN
 F 1 "10u" H 3425 1050 50  0000 L CNN
-F 2 "Capacitors_SMD:C_1206" H 3438 1000 50  0001 C CNN
+F 2 "CE_Capacitor:C_1206" H 3438 1000 50  0001 C CNN
 F 3 "" H 3400 1150 50  0000 C CNN
 	1    3400 1150

Commit message: CC58
Parts:
- removed C101: .1uf, CE_Capacitor:C_0805, symbol C
- removed C102, C103: 18pf, CE_Capacitor:C_0805, symbol C
- removed C104, C107: 0.1u, CE_Capacitor:C_0805, symbol C
- removed C105, C108: 1u, CE_Capacitor:C_1206, symbol C
- removed C106, C109: 10u, CE_Capacitor:C_1206, symbol C
- removed L101: 10uh, CE_Inductor:Neosid_Inductor_SM1206, symbol INDUCTOR
- removed P107, P108, P109, P110: CONN_01X01, CE_MountingHole:MountingHole_3mm, symbol CONN_01X01
- removed Y101: Crystal, CE_Crystal:Crystal_HC49_US, symbol Crystal
- added C101, C104, C107: 08055C104JAT2A, CE_Capacitor:C_0805, symbol 08055C104JAT2A
- added C102, C103: 08055A180JAT2A, CE_Capacitor:C_0805, symbol 08055A180JAT2A
- added C105, C108: C1206C105M4RACTU, CE_Capacitor:C_1206, symbol C1206C105M4RACTU
- added C106, C109: CC1206KKX7R8BB106, CE_Capacitor:C_1206, symbol CC1206KKX7R8BB106
- added L101: AIML-1206-100K-T, CE_Inductor:Neosid_Inductor_SM1206, symbol AIML-1206-100K-T
- added P107, P108, P109, P110: 3MM_HOLE, CE_MountingHole:MountingHole_3mm, symbol 3MM_HOLE
- added Y101: 9C-8.000MEEJ-T, CE_Crystal:Crystal_HC49_US, symbol 9C-8.000MEEJ-T
Connections:
- net GND: now also C101.2, C102.1, C103.1, C104.2, C105.2, C106.2, C107.2, C108.2, C109.2
- net PWR: now also C104.1, C105.1, C106.1, C107.1, C108.1, C109.1, L101.1
- net VDDA: now also C101.1, L101.2
- net at U101.5 (PF0-OSC_IN): now also C102.2, Y101.2
- net at U101.6 (PF1-OSC_OUT): now also C103.2, Y101.1
Other:
- note added: "2.9.2016 / 1.2.2017?"
- note added: "v2 ?"
- note removed: "2.9.2016"
- note removed: "v2"
