File: hardware/pcb/CentralCommand.kicad_pcb (KiCad board)
At the start: 4 copper layers, 53.3 x 73.1 mm, 72 parts, among them CON201 USB-MICRO-B, P101 CONN_01X10, P102 CONN_01X10, P103 CONN_01X04, P104 CONN_01X04, P105 CONN_01X02, P106 CONN_01X02, P107 CONN_01X01, P108 CONN_01X01, P109 CONN_01X01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

Commit message: CC56
Parts:
- C101, C102, C103, C104, C107, C201, C202, C204, C301, C302: footprint Capacitors_SMD:C_0805 -> CE_Capacitor:C_0805
- C105, C106, C108, C109: footprint Capacitors_SMD:C_1206 -> CE_Capacitor:C_1206
- C203, C205, C206: footprint Capacitors_SMD:C_1210 -> CE_Capacitor:C_1210
- CON201: footprint pcb:MICRO_B_CONN_10118193-0001LF -> CE_Connector:MICRO_B_CONN_10118193-0001LF
- D203, D204, D205: footprint LEDs:LED_0805 -> CE_Diode:LED_0805
- FB201, L101: footprint Inductors_NEOSID:Neosid_Inductor_SM1206 -> CE_Inductor:Neosid_Inductor_SM1206
- JP201, P305: footprint Pin_Headers:Pin_Header_Straight_1x03 -> CE_Connector:Pin_Header_Straight_1x03
- P101, P102: footprint Pin_Headers:Pin_Header_Straight_1x10 -> CE_Connector:Pin_Header_Straight_1x10
- P103, P104: footprint Pin_Headers:Pin_Header_Straight_1x04 -> CE_Connector:Pin_Header_Straight_1x04
- P105, P106, P202, P302: footprint Pin_Headers:Pin_Header_Straight_1x02 -> CE_Connector:Pin_Header_Straight_1x02
- P107, P108, P109, P110: footprint Mounting_Holes:MountingHole_3mm -> CE_MountingHole:MountingHole_3mm
- P301: footprint Pin_Headers:Pin_Header_Straight_1x06 -> CE_Connector:Pin_Header_Straight_1x06
- P303, P304: footprint pcb:GroveConnectorStraight_B4B-PH-K-S -> CE_Connector:GroveConnectorStraight_B4B-PH-K-S
- R201, R202, R203, R204, R205, R206, R207, R208, R209, R210, R211, R301, R302, R303, R304, R305, R306, R307, R308, R309, R310, R311, R312, R313: footprint Resistors_SMD:R_0805 -> CE_Resistor:R_0805
- U101: footprint Housings_QFP:LQFP-48_7x7mm_Pitch0.5mm -> CE_IC:LQFP-48_7x7mm_Pitch0.5mm
- U201: footprint Housings_DFN_QFN:QFN-32-1EP_5x5mm_Pitch0.5mm -> CE_IC:QFN-32-1EP_5x5mm_Pitch0.5mm
- U202: footprint pcb:SOT-23 -> CE_Regulator:SOT-23
- U301, U302: footprint pcb:Pushbutton_B3F-1020 -> CE_Switch:Pushbutton_B3F-1020
- Y101: footprint pcb:Crystal_HC49_US -> CE_Crystal:Crystal_HC49_US

Commit message: CC56
Parts:
- D201, D202: footprint Diodes_SMD:SOD-123 -> CE_Diode:SOD-123
Changed lines of the file:
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@@
     )
   )
-  (module Diodes_SMD:SOD-123 (layer F.Cu)
+  (module CE_Diode:SOD-123 (layer F.Cu)
     (at 53.5 95.5 270)
     (descr SOD-123)
@@
       (net 13 "Net-(D201-Pad2)"))
   )
-  (module Diodes_SMD:SOD-123 (layer F.Cu)
+  (module CE_Diode:SOD-123 (layer F.Cu)
     (at 53.7 87.25 90)
     (descr SOD-123)

Commit message: Re-reading the netlist in pcbnew broke the Front CU as KiCad has changed the sheet mapping of nets.  /comm/pwr became just /pwr.  I had to associate /pwr to the Front CU.
Parts:
- C101: value C -> .1uf
- D203: value LED -> LED_GREEN
- D204: value LED -> LED_YELLOW
- D205: value LED -> LED_BLUE
- L101: value INDUCTOR -> 10uh
- R305: value R -> 0
Connections:
- net /Comm/BOOT0 renamed /BOOT0
- net /Comm/MC0 renamed /MC0
- net /Comm/NRST renamed /NRST
- net /Comm/PWR renamed /PWR
- net /Comm/SCL renamed /I2C_SCL
- net /Comm/SDA renamed /I2C_SDA
- net /Comm/SWCLK renamed /SWCLK
- net /Comm/SWDIO renamed /SWDIO
- net /Comm/TRACE renamed /TRACE
- net /Comm/WKUP1 renamed /WKUP1
- net /Power/RXD renamed /USART2_RX
- net /Power/TXD renamed /USART2_TX

Commit message: CC58
Parts:
- C101: value .1uf -> 08055C104JAT2A
- C102, C103: value 18pf -> 08055A180JAT2A
- C104, C107: value 0.1u -> 08055C104JAT2A
- C105, C108: value 1u -> C1206C105M4RACTU
- C106, C109: value 10u -> CC1206KKX7R8BB106
- C201: value 10nf -> C0805C103K3RACTU
- C202, C204: value 100nf -> 08055C104JAT2A
- C203: value 4.7uf -> CL21B475KOFNNNE; footprint CE_Capacitor:C_1210 -> CE_Capacitor:C_0805
- C205, C206: value 10uf -> TMK325B7106KN-TR
- CON201: value USB-MICRO-B -> 10118193-0001LF
- D201, D202: value D_Schottky -> MBR0520LT1G
- D203: value LED_GREEN -> 150080GS75000
- D204: value LED_YELLOW -> 150080YS75000
- D205: value LED_BLUE -> 150080BS75000
- FB201: value FILTER -> BLM41PG471SN1L; footprint CE_Inductor:Neosid_Inductor_SM1206 -> CE_Filter:Filter_SM1806
- L101: value 10uh -> AIML-1206-100K-T
- P107, P108, P109, P110: value CONN_01X01 -> 3MM_HOLE
- R201, R202, R203, R205, R207: value 0 -> ERJ-6GEY0R00V
- R208, R209, R211: value 270 -> RNCP0805FTD200R
- Y101: value Crystal -> 9C-8.000MEEJ-T
Connections:
- R205 pad 2: /USART2_TX -> /USART2_RX
- R207 pad 2: /USART2_RX -> /USART2_TX
Routing:
- net /USART2_TX: track 21.2 -> 25.4 mm
- net /USART2_RX: track 21.8 -> 20.0 mm

Commit message: CC58
Parts:
- C301, C302: value 0.1uf -> C0805C104K3RACTU
- R301, R302, R305, R306, R307, R308, R309, R310, R311, R312, R313: value 0 -> ERJ-6GEY0R00V
- R303, R304: value 100k -> RMCF0805FT100K; footprint CE_Resistor:R_0805 -> CE_Capacitor:C_0805
Changed lines of the file:
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@@
       (effects (font (size 0.5 0.5) (thickness 0.125)))
     )
-    (fp_text value 0.1uf (at 0 2.1 270) (layer F.Fab)
+    (fp_text value C0805C104K3RACTU (at 0 2.1 270) (layer F.Fab)
       (effects (font (size 0.5 0.5) (thickness 0.125)))
     )
@@
       (effects (font (size 0.5 0.5) (thickness 0.125)))
     )
-    (fp_text value 0.1uf (at 0 2.1 270) (layer F.Fab)
+    (fp_text value C0805C104K3RACTU (at 0 2.1 270) (layer F.Fab)
       (effects (font (size 0.5 0.5) (thickness 0.125)))
     )
@@
       (effects (font (size 0.5 0.5) (thickness 0.125)))
     )
-    (fp_text value 0 (at 0 2.1) (layer F.Fab)
+    (fp_text value ERJ-6GEY0R00V (at 0 2.1) (layer F.Fab)
       (effects (font (size 0.5 0.5) (thickness 0.125)))
     )
@@
       (effects (font (size 0.5 0.5) (thickness 0.125)))
     )
-    (fp_text value 0 (at 0 2.1 270) (layer F.Fab)
+    (fp_text value ERJ-6GEY0R00V (at 0 2.1 270) (layer F.Fab)
       (effects (font (size 0.5 0.5) (thickness 0.125)))
     )
@@
   )
   (module CE_Resistor:R_0805 (layer F.Cu)
-    (at 93.84 53.38 270)
-    (descr "Resistor SMD 0805, reflow soldering, Vishay (see dcrcw.pdf)")
-    (tags "resistor 0805")
-    (attr smd)
-    (fp_text reference R303 (at -2.05 -0.04 360) (layer F.SilkS)
-      (effects (font (size 0.5 0.5) (thickness 0.125)))
-    )
-    (fp_text value 100k (at 0 2.1 270) (layer F.Fab)
-      (effects (font (size 0.5 0.5) (thickness 0.125)))
-    )
-    (fp_line (start -1.6 -1) (end 1.6 -1) (layer F.CrtYd) (width 0.05))
-    (fp_line (start -1.6 1) (end 1.6 1) (layer F.CrtYd) (width 0.05))
-    (fp_line (start -1.6 -1) (end -1.6 1) (layer F.CrtYd) (width 0.05))
-    (fp_line (start 1.6 -1) (end 1.6 1) (layer F.CrtYd) (width 0.05))
-    (fp_line (start 0.6 0.875) (end -0.6 0.875) (layer F.SilkS) (width 0.15))
-    (fp_line (start -0.6 -0.875) (end 0.6 -0.875) (layer F.SilkS) (width 0.15))
-    (pad 1 smd rect (at -0.95 0 270) (size 0.7 1.3) (layers F.Cu F.Paste F.Mask)
-      (net 87 /PWR))
-    (pad 2 smd rect (at 0.95 0 270) (size 0.7 1.3) (layers F.Cu F.Paste F.Mask)
-      (net 91 /SWDIO))
-    (model ${KIPRJMOD}/../CE_KiCad_Lib/packages3d/CE_Resistor.3dshapes/R_0805.wrl
-      (at (xyz 0 0 0))
-      (scale (xyz 1 1 1))
-      (rotate (xyz 0 0 0))
-    )
-  )
-  (module CE_Resistor:R_0805 (layer F.Cu)
-    (at 93.46 57 90)
-    (descr "Resistor SMD 0805, reflow soldering, Vishay (see dcrcw.pdf)")
-    (tags "resistor 0805")
-    (attr smd)
-    (fp_text reference R304 (at -2.06 0 180) (layer F.SilkS)
-      (effects (font (size 0.5 0.5) (thickness 0.125)))
-    )
-    (fp_text value 100k (at 0 2.1 90) (layer F.Fab)
-      (effects (font (size 0.5 0.5) (thickness 0.125)))
-    )
-    (fp_line (start -1.6 -1) (end 1.6 -1) (layer F.CrtYd) (width 0.05))
-    (fp_line (start -1.6 1) (end 1.6 1) (layer F.CrtYd) (width 0.05))
-    (fp_line (start -1.6 -1) (end -1.6 1) (layer F.CrtYd) (width 0.05))
-    (fp_line (start 1.6 -1) (end 1.6 1) (layer F.CrtYd) (width 0.05))
-    (fp_line (start 0.6 0.875) (end -0.6 0.875) (layer F.SilkS) (width 0.15))
-    (fp_line (start -0.6 -0.875) (end 0.6 -0.875) (layer F.SilkS) (width 0.15))
-    (pad 1 smd rect (at -0.95 0 90) (size 0.7 1.3) (layers F.Cu F.Paste F.Mask)
-      (net 90 /SWCLK))
-    (pad 2 smd rect (at 0.95 0 90) (size 0.7 1.3) (layers F.Cu F.Paste F.Mask)
-      (net 1 GND))
-    (model ${KIPRJMOD}/../CE_KiCad_Lib/packages3d/CE_Resistor.3dshapes/R_0805.wrl
-      (at (xyz 0 0 0))
-      (scale (xyz 1 1 1))
-      (rotate (xyz 0 0 0))
-    )
-  )
-  (module CE_Resistor:R_0805 (layer F.Cu)
     (at 89.03 62.74)
     (descr "Resistor SMD 0805, reflow soldering, Vishay (see dcrcw.pdf)")
@@
       (effects (font (size 0.5 0.5) (thickness 0.125)))
     )
-    (fp_text value 0 (at 0 2.1) (layer F.Fab)
+    (fp_text value ERJ-6GEY0R00V (at 0 2.1) (layer F.Fab)
       (effects (font (size 0.5 0.5) (thickness 0.125)))
     )
@@
       (effects (font (size 0.5 0.5) (thickness 0.125)))
     )
-    (fp_text value 0 (at 0 2.1 90) (layer F.Fab)
+    (fp_text value ERJ-6GEY0R00V (at 0 2.1 90) (layer F.Fab)
       (effects (font (size 0.5 0.5) (thickness 0.125)))
     )
@@
       (effects (font (size 0.5 0.5) (thickness 0.125)))
     )
-    (fp_text value 0 (at 0 2.1 90) (layer F.Fab)
+    (fp_text value ERJ-6GEY0R00V (at 0 2.1 90) (layer F.Fab)
       (effects (font (size 0.5 0.5) (thickness 0.125)))
     )
@@
       (effects (font (size 0.5 0.5) (thickness 0.125)))
     )
-    (fp_text value 0 (at 0 2.1 90) (layer F.Fab)
+    (fp_text value ERJ-6GEY0R00V (at 0 2.1 90) (layer F.Fab)
       (effects (font (size 0.5 0.5) (thickness 0.125)))
     )
@@
       (effects (font (size 0.5 0.5) (thickness 0.125)))
     )
-    (fp_text value 0 (at 0 2.1 90) (layer F.Fab)
+    (fp_text value ERJ-6GEY0R00V (at 0 2.1 90) (layer F.Fab)
       (effects (font (size 0.5 0.5) (thickness 0.125)))
     )
@@
       (effects (font (size 0.5 0.5) (thickness 0.125)))
     )
-    (fp_text value 0 (at 0 2.1 270) (layer F.Fab)
+    (fp_text value ERJ-6GEY0R00V (at 0 2.1 270) (layer F.Fab)
       (effects (font (size 0.5 0.5) (thickness 0.125)))
     )
@@
       (effects (font (size 0.5 0.5) (thickness 0.125)))
     )
-    (fp_text value 0 (at 0 2.1 270) (layer F.Fab)
+    (fp_text value ERJ-6GEY0R00V (at 0 2.1 270) (layer F.Fab)
       (effects (font (size 0.5 0.5) (thickness 0.125)))
     )
@@
       (effects (font (size 0.5 0.5) (thickness 0.125)))
     )
-    (fp_text value 0 (at 0 2.1 270) (layer F.Fab)
+    (fp_text value ERJ-6GEY0R00V (at 0 2.1 270) (layer F.Fab)
       (effects (font (size 0.5 0.5) (thickness 0.125)))
     )
@@
       (effects (font (size 0.5 0.5) (thickness 0.125)))
     )
-    (fp_text value 0 (at 0 2.1 270) (layer F.Fab)
+    (fp_text value ERJ-6GEY0R00V (at 0 2.1 270) (layer F.Fab)
       (effects (font (size 0.5 0.5) (thickness 0.125)))
     )
@@
     (model ${KIPRJMOD}/../CE_KiCad_Lib/packages3d/CE_Capacitor.3dshapes/C_0805.wrl
       (at (xyz 0 0 0))
+      (scale (xyz 1 1 1))
+      (rotate (xyz 0 0 0))
+    )
+  )
+  (module CE_Capacitor:C_0805 (layer F.Cu)
+    (at 93.84 53.38 270)
+    (descr "Capacitor SMD 0805, reflow soldering, AVX (see smccp.pdf)")
+    (tags "capacitor 0805")
+    (attr smd)
+    (fp_text reference R303 (at -0.53 1.49 270) (layer F.SilkS)
+      (effects (font (size 0.5 0.5) (thickness 0.125)))
+    )
+    (fp_text value RMCF0805FT100K (at 0 2.1 270) (layer F.Fab)
+      (effects (font (size 1 1) (thickness 0.15)))
+    )
+    (fp_line (start -1 0.625) (end -1 -0.625) (layer F.Fab) (width 0.15))
+    (fp_line (start 1 0.625) (end -1 0.625) (layer F.Fab) (width 0.15))
+    (fp_line (start 1 -0.625) (end 1 0.625) (layer F.Fab) (width 0.15))
+    (fp_line (start -1 -0.625) (end 1 -0.625) (layer F.Fab) (width 0.15))
+    (fp_line (start -1.8 -1) (end 1.8 -1) (layer F.CrtYd) (width 0.05))
+    (fp_line (start -1.8 1) (end 1.8 1) (layer F.CrtYd) (width 0.05))
+    (fp_line (start -1.8 -1) (end -1.8 1) (layer F.CrtYd) (width 0.05))
+    (fp_line (start 1.8 -1) (end 1.8 1) (layer F.CrtYd) (width 0.05))
+    (fp_line (start 0.5 -0.85) (end -0.5 -0.85) (layer F.SilkS) (width 0.15))
+    (fp_line (start -0.5 0.85) (end 0.5 0.85) (layer F.SilkS) (width 0.15))
+    (pad 1 smd rect (at -1 0 270) (size 1 1.25) (layers F.Cu F.Paste F.Mask)
+      (net 87 /PWR))
+    (pad 2 smd rect (at 1 0 270) (size 1 1.25) (layers F.Cu F.Paste F.Mask)
+      (net 91 /SWDIO))
+    (model ${KIPRJMOD}/../CE_KiCad_Lib/packages3d/CE_Capacitor.3dshapes/C_0805.wrl
+      (at (xyz 0 0 0))
+      (scale (xyz 1 1 1))
+      (rotate (xyz 0 0 0))
+    )
+  )
+  (module CE_Capacitor:C_0805 (layer F.Cu)
+    (at 93.46 57 90)
+    (descr "Capacitor SMD 0805, reflow soldering, AVX (see smccp.pdf)")
+    (tags "capacitor 0805")
+    (attr smd)
+    (fp_text reference R304 (at 0.2 -1.435 90) (layer F.SilkS)
+      (effects (font (size 0.5 0.5) (thickness 0.125)))
+    )
+    (fp_text value RMCF0805FT100K (at 0 2.1 90) (layer F.Fab)
+      (effects (font (size 1 1) (thickness 0.15)))
+    )
+    (fp_line (start -1 0.625) (end -1 -0.625) (layer F.Fab) (width 0.15))
+    (fp_line (start 1 0.625) (end -1 0.625) (layer F.Fab) (width 0.15))
+    (fp_line (start 1 -0.625) (end 1 0.625) (layer F.Fab) (width 0.15))
+    (fp_line (start -1 -0.625) (end 1 -0.625) (layer F.Fab) (width 0.15))
+    (fp_line (start -1.8 -1) (end 1.8 -1) (layer F.CrtYd) (width 0.05))
+    (fp_line (start -1.8 1) (end 1.8 1) (layer F.CrtYd) (width 0.05))
+    (fp_line (start -1.8 -1) (end -1.8 1) (layer F.CrtYd) (width 0.05))
+    (fp_line (start 1.8 -1) (end 1.8 1) (layer F.CrtYd) (width 0.05))
+    (fp_line (start 0.5 -0.85) (end -0.5 -0.85) (layer F.SilkS) (width 0.15))
+    (fp_line (start -0.5 0.85) (end 0.5 0.85) (layer F.SilkS) (width 0.15))
+    (pad 1 smd rect (at -1 0 90) (size 1 1.25) (layers F.Cu F.Paste F.Mask)
+      (net 90 /SWCLK))
+    (pad 2 smd rect (at 1 0 90) (size 1 1.25) (layers F.Cu F.Paste F.Mask)
+      (net 1 GND))
+    (model ${KIPRJMOD}/../CE_KiCad_Lib/packages3d/CE_Capacitor.3dshapes/C_0805.wrl
+      (at (xyz 0 0 0))
