File: hardware/pcb/Comm.sch (KiCad schematic (older format))
At the start: 22 parts, among them P301 CONN_01X06, P302 CONN_01X02, P303 CONN_01X04, P304 CONN_01X04, P305 CONN_01X03, U301 B3F-1020, U302 B3F-1020

Commit message: CC56
Parts:
- C301, C302: footprint Capacitors_SMD:C_0805 -> CE_Capacitor:C_0805
- P301: footprint Pin_Headers:Pin_Header_Straight_1x06 -> CE_Connector:Pin_Header_Straight_1x06
- P302: footprint Pin_Headers:Pin_Header_Straight_1x02 -> CE_Connector:Pin_Header_Straight_1x02
- P303, P304: footprint pcb:GroveConnectorStraight_B4B-PH-K-S -> CE_Connector:GroveConnectorStraight_B4B-PH-K-S
- P305: footprint Pin_Headers:Pin_Header_Straight_1x03 -> CE_Connector:Pin_Header_Straight_1x03
- R301, R302, R303, R304, R305, R306, R307, R308, R309, R310, R311, R312, R313: footprint Resistors_SMD:R_0805 -> CE_Resistor:R_0805
- U301, U302: footprint pcb:Pushbutton_B3F-1020 -> CE_Switch:Pushbutton_B3F-1020
Changed lines of the file:
@@
 F 0 "P303" H 6100 2550 50  0000 C CNN
 F 1 "CONN_01X04" V 6200 2300 50  0000 C CNN
-F 2 "pcb:GroveConnectorStraight_B4B-PH-K-S" H 6100 2300 50  0001 C CNN
+F 2 "CE_Connector:GroveConnectorStraight_B4B-PH-K-S" H 6100 2300 50  0001 C CNN
 F 3 "" H 6100 2300 50  0000 C CNN
 F 4 "S4B-PH-K-S(LF)(SN)" H 6100 2300 60  0001 C CNN "MPN"
@@
 F 0 "P304" H 5650 4050 50  0000 C CNN
 F 1 "CONN_01X04" V 5750 3800 50  0000 C CNN
-F 2 "pcb:GroveConnectorStraight_B4B-PH-K-S" H 5650 3800 50  0001 C CNN
+F 2 "CE_Connector:GroveConnectorStraight_B4B-PH-K-S" H 5650 3800 50  0001 C CNN
 F 3 "" H 5650 3800 50  0000 C CNN
 F 4 "S4B-PH-K-S(LF)(SN)" H 5650 3800 60  0001 C CNN "MPN"
@@
 F 0 "P301" H 900 5550 50  0000 C CNN
 F 1 "CONN_01X06" V 1000 5200 50  0000 C CNN
-F 2 "Pin_Headers:Pin_Header_Straight_1x06" H 900 5200 50  0001 C CNN
+F 2 "CE_Connector:Pin_Header_Straight_1x06" H 900 5200 50  0001 C CNN
 F 3 "" H 900 5200 50  0000 C CNN
 	1    900  5200
@@
 F 0 "R301" V 1230 4650 50  0000 C CNN
 F 1 "0" V 1150 4650 50  0000 C CNN
-F 2 "Resistors_SMD:R_0805" V 1080 4650 50  0001 C CNN
+F 2 "CE_Resistor:R_0805" V 1080 4650 50  0001 C CNN
 F 3 "" H 1150 4650 50  0000 C CNN
 	1    1150 4650
@@
 F 0 "R303" V 1480 4650 50  0000 C CNN
 F 1 "100k" V 1400 4650 50  0000 C CNN
-F 2 "Resistors_SMD:R_0805" V 1330 4650 50  0001 C CNN
+F 2 "CE_Resistor:R_0805" V 1330 4650 50  0001 C CNN
 F 3 "" H 1400 4650 50  0000 C CNN
 	1    1400 4650
@@
 F 0 "R304" V 1980 5350 50  0000 C CNN
 F 1 "100k" V 1900 5350 50  0000 C CNN
-F 2 "Resistors_SMD:R_0805" V 1830 5350 50  0001 C CNN
+F 2 "CE_Resistor:R_0805" V 1830 5350 50  0001 C CNN
 F 3 "" H 1900 5350 50  0000 C CNN
 	1    1900 5350
@@
 F 0 "R302" V 1280 5750 50  0000 C CNN
 F 1 "0" V 1200 5750 50  0000 C CNN
-F 2 "Resistors_SMD:R_0805" V 1130 5750 50  0001 C CNN
+F 2 "CE_Resistor:R_0805" V 1130 5750 50  0001 C CNN
 F 3 "" H 1200 5750 50  0000 C CNN
 	1    1200 5750
@@
 F 0 "C301" H 975 7050 50  0000 L CNN
 F 1 "0.1uf" H 975 6850 50  0000 L CNN
-F 2 "Capacitors_SMD:C_0805" H 988 6800 50  0001 C CNN
+F 2 "CE_Capacitor:C_0805" H 988 6800 50  0001 C CNN
 F 3 "" H 950 6950 50  0000 C CNN
 	1    950  6950
@@
 F 0 "C302" H 2425 7050 50  0000 L CNN
 F 1 "0.1uf" H 2425 6850 50  0000 L CNN
-F 2 "Capacitors_SMD:C_0805" H 2438 6800 50  0001 C CNN
+F 2 "CE_Capacitor:C_0805" H 2438 6800 50  0001 C CNN
 F 3 "" H 2400 6950 50  0000 C CNN
 	1    2400 6950
@@
 F 0 "R305" V 4030 6950 50  0000 C CNN
 F 1 "0" V 3950 6950 50  0000 C CNN
-F 2 "Resistors_SMD:R_0805" V 3880 6950 50  0001 C CNN
+F 2 "CE_Resistor:R_0805" V 3880 6950 50  0001 C CNN
 F 3 "" H 3950 6950 50  0000 C CNN
 	1    3950 6950
@@
 F 0 "P302" H 3450 7150 50  0000 C CNN
 F 1 "CONN_01X02" V 3600 7000 50  0000 C CNN
-F 2 "Pin_Headers:Pin_Header_Straight_1x02" H 3450 7000 50  0001 C CNN
+F 2 "CE_Connector:Pin_Header_Straight_1x02" H 3450 7000 50  0001 C CNN
 F 3 "" H 3450 7000 50  0000 C CNN
 	1    3450 7000
@@
 F 0 "P305" H 5000 7150 50  0000 C CNN
 F 1 "CONN_01X03" V 5150 6950 50  0000 C CNN
-F 2 "Pin_Headers:Pin_Header_Straight_1x03" H 5000 6950 50  0001 C CNN
+F 2 "CE_Connector:Pin_Header_Straight_1x03" H 5000 6950 50  0001 C CNN
 F 3 "" H 5000 6950 50  0000 C CNN
 	1    5000 6950
@@
 F 0 "U301" V 1400 6600 60  0000 C CNN
 F 1 "B3F-1020" V 1250 6900 60  0000 C CNN
-F 2 "pcb:Pushbutton_B3F-1020" H 1350 6900 60  0001 C CNN
+F 2 "CE_Switch:Pushbutton_B3F-1020" H 1350 6900 60  0001 C CNN
 F 3 "" H 1350 6900 60  0000 C CNN
 F 4 "B3F-1020" H 1350 6900 60  0001 C CNN "MPN"
@@
 F 0 "U302" V 2850 6600 60  0000 C CNN
 F 1 "B3F-1020" V 2700 6950 60  0000 C CNN
-F 2 "pcb:Pushbutton_B3F-1020" H 2800 6950 60  0001 C CNN
+F 2 "CE_Switch:Pushbutton_B3F-1020" H 2800 6950 60  0001 C CNN
 F 3 "" H 2800 6950 60  0000 C CNN
 F 4 "B3F-1020" H 2800 6950 60  0001 C CNN "MPN"
@@
 F 0 "R310" V 5730 1950 50  0000 C CNN
 F 1 "0" V 5650 1950 50  0000 C CNN
-F 2 "Resistors_SMD:R_0805" V 5580 1950 50  0001 C CNN
+F 2 "CE_Resistor:R_0805" V 5580 1950 50  0001 C CNN
 F 3 "" H 5650 1950 50  0000 C CNN
 	1    5650 1950
@@
 F 0 "R311" V 5730 2150 50  0000 C CNN
 F 1 "0" V 5650 2150 50  0000 C CNN
-F 2 "Resistors_SMD:R_0805" V 5580 2150 50  0001 C CNN
+F 2 "CE_Resistor:R_0805" V 5580 2150 50  0001 C CNN
 F 3 "" H 5650 2150 50  0000 C CNN
 	1    5650 2150
@@
 F 0 "R313" V 5730 2550 50  0000 C CNN
 F 1 "0" V 5650 2550 50  0000 C CNN
-F 2 "Resistors_SMD:R_0805" V 5580 2550 50  0001 C CNN
+F 2 "CE_Resistor:R_0805" V 5580 2550 50  0001 C CNN
 F 3 "" H 5650 2550 50  0000 C CNN
 	1    5650 2550
@@
 F 0 "R312" V 5730 2350 50  0000 C CNN
 F 1 "0" V 5650 2350 50  0000 C CNN
-F 2 "Resistors_SMD:R_0805" V 5580 2350 50  0001 C CNN
+F 2 "CE_Resistor:R_0805" V 5580 2350 50  0001 C CNN
 F 3 "" H 5650 2350 50  0000 C CNN
 	1    5650 2350
@@
 F 0 "R309" V 5280 4100 50  0000 C CNN
 F 1 "0" V 5200 4100 50  0000 C CNN
-F 2 "Resistors_SMD:R_0805" V 5130 4100 50  0001 C CNN
+F 2 "CE_Resistor:R_0805" V 5130 4100 50  0001 C CNN
 F 3 "" H 5200 4100 50  0000 C CNN
 	1    5200 4100
@@
 F 0 "R308" V 5280 3900 50  0000 C CNN
 F 1 "0" V 5200 3900 50  0000 C CNN
-F 2 "Resistors_SMD:R_0805" V 5130 3900 50  0001 C CNN
+F 2 "CE_Resistor:R_0805" V 5130 3900 50  0001 C CNN
 F 3 "" H 5200 3900 50  0000 C CNN
 	1    5200 3900
@@
 F 0 "R307" V 5280 3700 50  0000 C CNN
 F 1 "0" V 5200 3700 50  0000 C CNN
-F 2 "Resistors_SMD:R_0805" V 5130 3700 50  0001 C CNN
+F 2 "CE_Resistor:R_0805" V 5130 3700 50  0001 C CNN
 F 3 "" H 5200 3700 50  0000 C CNN
 	1    5200 3700
@@
 F 0 "R306" V 5280 3500 50  0000 C CNN
 F 1 "0" V 5200 3500 50  0000 C CNN
-F 2 "Resistors_SMD:R_0805" V 5130 3500 50  0001 C CNN
+F 2 "CE_Resistor:R_0805" V 5130 3500 50  0001 C CNN
 F 3 "" H 5200 3500 50  0000 C CNN
 	1    5200 3500

Commit message: CC58
Parts:
- removed C301, C302: 0.1uf, CE_Capacitor:C_0805, symbol C
- removed R301, R302, R305, R306, R307, R308, R309, R310, R311, R312, R313: 0, CE_Resistor:R_0805, symbol R
- removed R303, R304: 100k, CE_Resistor:R_0805, symbol R
- added C301, C302: C0805C104K3RACTU, CE_Capacitor:C_0805, symbol C0805C104K3RACTU
- added R301, R302, R305, R306, R307, R308, R309, R310, R311, R312, R313: ERJ-6GEY0R00V, CE_Resistor:R_0805, symbol ERJ-6GEY0R00V
- added R303, R304: RMCF0805FT100K, CE_Capacitor:C_0805, symbol RMCF0805FT100K
Connections:
- net CLOCKOUT: now also R305.2
- net GND: now also C301.2, C302.2, R304.2, R306.2, R310.2
- net MC0: now also R305.1
- net NRST: now also C301.1
- net PWR: now also R301.1, R303.1, R307.2, R311.2
- net SCL: now also R308.2, R312.2
- net SDA: now also R309.2, R313.2
- net SWCLK: now also R304.1
- net SWDIO: now also R303.2
- net TRACE: now also R302.2
- net WKUP1: now also C302.1
- net at P303.1 (P1): now also R310.1
- net at P303.2 (P2): now also R311.1
- net at P303.3 (P3): now also R312.1
- net at P303.4 (P4): now also R313.1
- net at P304.1 (P1): now also R306.1
- net at P304.2 (P2): now also R307.1
- net at P304.3 (P3): now also R308.1
- net at P304.4 (P4): now also R309.1
- net at P301.1 (P1): now also R301.2
- net at P301.6 (P6): now also R302.1
Other:
- moved on the sheet: P304
